Commit message: fixed inertia values in urdf

File: urdf/mico_simplified.URDF (robot description, URDF)
Before this commit: robot mico_simplified, 13 links, 12 joints
Links:
- link Finger_1_Distal_Link: mass 0.0121939442358921 -> 0.4
- link Finger_1_Proximal_Link: mass 0.0106365214895162 -> 0.4
- link Finger_2_Distal_Link: mass 0.012193944229752 -> 0.4
- link Finger_2_Proximal_Link: mass 0.0106365251828778 -> 0.4
Joints:
- joint Arm_Joint: limit lower=-2.26 upper=2.26 effort=0 velocity=0 -> lower=-2.26 upper=2.26 effort=1000 velocity=1
- joint Finger_1_Distal_Joint: limit lower=0 upper=0.78 effort=0 velocity=0 -> lower=-0.001 upper=0.78 effort=100 velocity=1
- joint Finger_1_Proximal_Joint: limit lower=0 upper=0.78 effort=0 velocity=0 -> lower=-0.001 upper=0.78 effort=100 velocity=1
- joint Finger_2_Distal_Joint: limit lower=0 upper=0.78 effort=0 velocity=0 -> lower=-0.01 upper=0.78 effort=100 velocity=.2
- joint Finger_2_Proximal_Joint: limit lower=0 upper=0.78 effort=0 velocity=0 -> lower=-0.001 upper=0.78 effort=100 velocity=1
- joint Forearm_Joint: limit lower=-2.44 upper=2.44 effort=0 velocity=0 -> lower=-2.44 upper=2.44 effort=1000 velocity=1
- joint Hand_Joint: limit lower=-3.14 upper=3.14 effort=0 velocity=0 -> lower=-3.14 upper=3.14 effort=1000 velocity=1
- joint Shoulder_Joint: limit lower=-3.14 upper=3.14 effort=0 velocity=0 -> lower=-3.14 upper=3.14 effort=1000 velocity=1
- joint Wrist_1_Joint: limit lower=-3.14 upper=3.14 effort=0 velocity=0 -> lower=-3.14 upper=3.14 effort=1000 velocity=10
- joint Wrist_2_Joint: limit lower=-3.14 upper=3.14 effort=0 velocity=0 -> lower=-3.14 upper=3.14 effort=1000 velocity=10
